File: Design Files/DZ/STM32_prj/V1I1/STM32/STM32.kicad_sch (KiCad schematic)
At the start: 0 parts

Commit message: Update 02
SCH and PCB Design
Parts:
- added C1, C12, C13, C19, C2, C3, C4, C5, C6, C8: 100n, Capacitor_SMD:C_0402_1005Metric, symbol Device:C
- added C10, C11, C14, C7, C9: 4u7, Capacitor_SMD:C_0603_1608Metric, symbol Device:C
- added C15: 0p8, Capacitor_SMD:C_0402_1005Metric, symbol Device:C
- added C16: 0p3, Capacitor_SMD:C_0402_1005Metric, symbol Device:C
- added C17, C18: 10p, Capacitor_SMD:C_0402_1005Metric, symbol Device:C
- added D1: LED, LED_SMD:LED_0402_1005Metric, symbol Device:LED
- added FLT1: DLF162500LT-5028A1, STM32_Footprint:DLF162500LT-5028A1, symbol STM32_sch_symbols:DLF162500LT-5028A1
- added J1: Conn_01x04, Connector_Molex:Molex_PicoBlade_53048-0410_1x04_P1.25mm_Horizontal, symbol Connector_Generic:Conn_01x04
- added J2: Conn_Coaxial, Connector_Coaxial:U.FL_Hirose_U.FL-R-SMT-1_Vertical, symbol Connector:Conn_Coaxial
- added J3: USB_C_Receptacle_USB2.0_16P, Connector_USB:USB_C_Receptacle_GCT_USB4105-xx-A_16P_TopMnt_Horizontal, symbol Connector:USB_C_Receptacle_USB2.0_16P
- added J4: Conn_ARM_SWD_TagConnect_TC2030, Connector:Tag-Connect_TC2030-IDC-FP_2x03_P1.27mm_Vertical, symbol Connector:Conn_ARM_SWD_TagConnect_TC2030
- added L1: 10n, Inductor_SMD:L_0402_1005Metric, symbol Device:L
- added L2: 10u, Inductor_SMD:L_0805_2012Metric, symbol Device:L
- added L3: 2n7, Inductor_SMD:L_0402_1005Metric, symbol Device:L
- added R1, R2, R3, R6: 220R, Resistor_SMD:R_0402_1005Metric, symbol Device:R
- added R4, R5, R7: 5k1, Resistor_SMD:R_0402_1005Metric, symbol Device:R
- added SW1: SW_Push, Button_Switch_SMD:SW_SPST_CK_RS282G05A3, symbol Switch:SW_Push
- added U1: MIC5365-3.3YD5, Package_TO_SOT_SMD:SOT-23-5, symbol Regulator_Linear:MIC5365-3.3YD5
- added U2: USBLC6-2SC6, Package_TO_SOT_SMD:SOT-23-6, symbol Power_Protection:USBLC6-2SC6
- added U3: STM32WB55CEUx, Package_DFN_QFN:QFN-48-1EP_7x7mm_P0.5mm_EP5.6x5.6mm, symbol MCU_ST_STM32WB:STM32WB55CEUx
- added X1: 32MHz, Crystal:Crystal_SMD_2016-4Pin_2.0x1.6mm, symbol Device:Crystal_GND24
- added X2: 32kHz768, Crystal:Crystal_SMD_2012-2Pin_2.0x1.2mm, symbol Device:Crystal_Small
Connections:
- new net: J4.6 (SWO), U3.43 (PB3)
- new net: R6.1, SW1.1
- new net: D1.2 (A), U3.16 (PA7)
- new net: X1.2, X1.4
- new net: D1.1 (K), R3.2
- new net +3V3: C1.1, C11.1, C12.1, C2.1, C3.1, C4.1, C5.1, C6.1, C7.1, C8.1, C9.1, J1.1 (Pin_1), J4.1 (VCC), SW1.2, U1.5 (VOUT), U3.1 (VBAT), U3.20 (VDD), U3.23 (VDDRF), U3.34 (VDDSMPS), U3.35 (VDD), U3.40 (VDDUSB), U3.48 (VDD), U3.8 (VDDA)
- new net +5V: C10.1, J3.A4 (VBUS), J3.A9 (VBUS), J3.B4 (VBUS), J3.B9 (VBUS), U1.1 (VIN), U1.3 (EN), U2.5 (VBUS)
- new net BOOT: C19.1, R6.2, R7.2, U3.4 (PH3)
- new net GND: C1.2, C10.2, C11.2, C12.2, C13.2, C14.2, C15.2, C16.2, C17.2, C18.2, C19.2, C2.2, C3.2, C4.2, C5.2, C6.2, C7.2, C8.2, C9.2, FLT1.2 (GND), FLT1.4 (GND), J1.4 (Pin_4), J2.2 (Ext), J3.A1 (GND), J3.A12 (GND), J3.B1 (GND), J3.B12 (GND), J3.S1 (SHIELD), J4.5 (GND), R3.1, R4.1, R5.1, R7.1, U1.2 (GND), U2.2 (GND), U3.22 (VSSRF), U3.32 (VSSSMPS), U3.49 (VSS)
- new net HSE_IN: U3.25 (OSC_IN), X1.3
- new net HSE_OUT: U3.24 (OSC_OUT), X1.1
- new net LSE_IN: C18.1, U3.2 (PC14), X2.2
- new net LSE_OUT: C17.1, U3.3 (PC15), X2.1
- new net RF: C15.1, L3.1, U3.21 (RF1)
- new net RF_ANT: FLT1.3 (OUT), J2.1 (In)
- new net RF_MATCH: C16.1, FLT1.1 (IN), L3.2
- new net SMPSLX: L1.1, U3.33 (VLXSMPS)
- new net SMPSLXL: L1.2, L2.1
- new net SMPS_FB: C14.1, L2.2, U3.31 (VFBSMPS)
- new net SWD_CLK: J4.4 (SWCLK), U3.41 (PA14)
- new net SWD_DIO: J4.2 (SWDIO), U3.39 (PA13)
- new net SWD_NRST: C13.1, J4.3 (~{RESET}), U3.7 (NRST)
- new net UART_RX: R2.2, U3.12 (PA3)
- new net UART_RXC: J1.3 (Pin_3), R2.1
- new net UART_TX: R1.2, U3.11 (PA2)
- new net UART_TXC: J1.2 (Pin_2), R1.1
- new net USBC_CC1: J3.A5 (CC1), R5.2
- new net USBC_CC2: J3.B5 (CC2), R4.2
- new net USBC_D+: J3.A6 (D+), J3.B6 (D+), U2.1 (I/O1)
- new net USBC_D-: J3.A7 (D-), J3.B7 (D-), U2.6 (I/O1)
- new net USB_D+: U2.3 (I/O2), U3.38 (PA12)
- new net USB_D-: U2.4 (I/O2), U3.37 (PA11)
- no-connect marks 0 -> 21
Other:
- note added: "${TITLE}"
- note added: "+5V TO +3V3 LDO REGULATOR"
- note added: "BOOT SWITCH"
- note added: "DECOUPLING CAPACITORS"
- note added: "HSE (32MHz) Crystal"
- note added: "LSE (32.768kHz) Crystal"
- note added: "RF Front-End & u.FL Connector"
- note added: "STM32WB55 MCU"
- note added: "TAG CONNECT SWD HEADER"
- note added: "UART HEADER"
- note added: "USB_C CONNECTOR"
- title: (none) -> STM32WB BOARD

Commit message: Update 03
Project accomplished
Parts:
- added FID1, FID2, FID3: Fiducial, Fiducial:Fiducial_1mm_Mask2mm, symbol Mechanical:Fiducial
- added H1, H2, H3, H4: MountingHole_Pad, MountingHole:MountingHole_2.2mm_M2_Pad, symbol Mechanical:MountingHole_Pad
Connections:
- net GND: now also H1.1, H2.1, H3.1, H4.1
Other:
- note added: "FIDUCIAL MARKERS"
- note added: "MOUNTING HOLES"
