File: Design Files/DZ/STM32_prj/V1I1/STM32/STM32.kicad_pcb (KiCad board)
At the start: 2 copper layers, 65 x 56 mm, 5 parts, among them J1 GPIO

Commit message: Update 02
SCH and PCB Design
Parts:
- removed MH1, MH2, MH3, MH4: MountingHole_2.7mm_M2.5, MountingHole:MountingHole_2.7mm_M2.5
- added C1: 100n, Capacitor_SMD:C_0402_1005Metric, F.Cu at (148.5, 56.5)
- added C10: 4u7, Capacitor_SMD:C_0603_1608Metric, F.Cu at (134.0, 69.0)
- added C11: 4u7, Capacitor_SMD:C_0603_1608Metric, F.Cu at (134.0, 67.5)
- added C12: 100n, Capacitor_SMD:C_0402_1005Metric, F.Cu at (143.5, 59.5)
- added C13: 100n, Capacitor_SMD:C_0402_1005Metric, F.Cu at (142.5, 54.5)
- added C14: 4u7, Capacitor_SMD:C_0603_1608Metric, F.Cu at (163.5, 54.5)
- added C15: 0p8, Capacitor_SMD:C_0402_1005Metric, F.Cu at (169.7, 61.0)
- added C16: 0p3, Capacitor_SMD:C_0402_1005Metric, F.Cu at (169.7, 64.0)
- added C17: 10p, Capacitor_SMD:C_0402_1005Metric, F.Cu at (157.5, 54.5)
- added C18: 10p, Capacitor_SMD:C_0402_1005Metric, F.Cu at (152.5, 54.5)
- added C19: 100n, Capacitor_SMD:C_0402_1005Metric, F.Cu at (139.5, 69.0)
- added C2: 100n, Capacitor_SMD:C_0402_1005Metric, F.Cu at (148.5, 58.0)
- added C3: 100n, Capacitor_SMD:C_0402_1005Metric, F.Cu at (148.5, 59.5)
- added C4: 100n, Capacitor_SMD:C_0402_1005Metric, F.Cu at (148.5, 61.0)
- added C5: 100n, Capacitor_SMD:C_0402_1005Metric, F.Cu at (148.5, 62.5)
- added C6: 100n, Capacitor_SMD:C_0402_1005Metric, F.Cu at (143.5, 56.5)
- added C7: 4u7, Capacitor_SMD:C_0603_1608Metric, F.Cu at (148.1, 54.4)
- added C8: 100n, Capacitor_SMD:C_0402_1005Metric, F.Cu at (143.5, 58.0)
- added C9: 4u7, Capacitor_SMD:C_0603_1608Metric, F.Cu at (134.0, 66.0)
- added D1: LED, LED_SMD:LED_0402_1005Metric, F.Cu at (159.3, 67.0)
- added FLT1: DLF162500LT-5028A1, STM32_Footprint:DLF162500LT-5028A1, F.Cu at (172.1, 62.4)
- added J2: Conn_Coaxial, Connector_Coaxial:U.FL_Hirose_U.FL-R-SMT-1_Vertical, F.Cu at (176.0, 62.0)
- added J3: USB_C_Receptacle_USB2.0_16P, Connector_USB:USB_C_Receptacle_GCT_USB4105-xx-A_16P_TopMnt_Horizontal, F.Cu at (122.5, 61.0)
- added J4: Conn_ARM_SWD_TagConnect_TC2030, Connector:Tag-Connect_TC2030-IDC-FP_2x03_P1.27mm_Vertical, F.Cu at (136.5, 59.6)
- added L1: 10n, Inductor_SMD:L_0402_1005Metric, F.Cu at (170.2, 56.0)
- added L2: 10u, Inductor_SMD:L_0805_2012Metric, F.Cu at (169.7, 54.5)
- added L3: 2n7, Inductor_SMD:L_0402_1005Metric, F.Cu at (170.2, 62.5)
- added R1: 220R, Resistor_SMD:R_0402_1005Metric, F.Cu at (157.1, 66.6)
- added R2: 220R, Resistor_SMD:R_0402_1005Metric, F.Cu at (157.1, 64.2)
- added R3: 220R, Resistor_SMD:R_0402_1005Metric, F.Cu at (159.3, 69.2)
- added R4: 5k1, Resistor_SMD:R_0402_1005Metric, F.Cu at (127.0, 67.0)
- added R5: 5k1, Resistor_SMD:R_0402_1005Metric, F.Cu at (126.5, 55.0)
- added R6: 220R, Resistor_SMD:R_0402_1005Metric, F.Cu at (139.5, 66.0)
- added R7: 5k1, Resistor_SMD:R_0402_1005Metric, F.Cu at (139.5, 67.5)
- added SW1: SW_Push, Button_Switch_SMD:SW_SPST_CK_RS282G05A3, F.Cu at (154.0, 64.5)
- added U1: MIC5365-3.3YD5, Package_TO_SOT_SMD:SOT-23-5, F.Cu at (130.0, 57.0)
- added U2: USBLC6-2SC6, Package_TO_SOT_SMD:SOT-23-6, F.Cu at (130.0, 64.0)
- added U3: STM32WB55CEUx, Package_DFN_QFN:QFN-48-1EP_7x7mm_P0.5mm_EP5.6x5.6mm, F.Cu at (163.0, 61.5)
- added X1: 32MHz, Crystal:Crystal_SMD_2016-4Pin_2.0x1.6mm, F.Cu at (166.5, 68.0)
- added X2: 32kHz768, Crystal:Crystal_SMD_2012-2Pin_2.0x1.2mm, F.Cu at (156.5, 57.5)
- J1: value GPIO -> Conn_01x04; footprint Connector_PinSocket_2.54mm:PinSocket_2x20_P2.54mm_Vertical -> Connector_Molex:Molex_PicoBlade_53048-0410_1x04_P1.25mm_Horizontal; moved to F.Cu
- moved J1 56.2 mm to (149.3, 68.2), turned to 180 degrees
Connections:
- J1 pad 2: +5V -> /UART_TXC
- J1 pad 3: /GPIO2/SDA1 -> /UART_RXC
- J1 pad 4: +5V -> GND
Routing:
- net GND: track 0.00 -> 82.1 mm, vias 0 -> 41
- net +3V3: track 0.00 -> 68.9 mm, vias 0 -> 15
- net /USB_D+: track 0.00 -> 47.4 mm, vias 0 -> 2
- net /SWD_DIO: track 0.00 -> 43.2 mm, vias 0 -> 2
- net /USB_D-: track 0.00 -> 42.7 mm, vias 0 -> 2
- net /SWD_NRST: track 0.00 -> 42.1 mm, vias 0 -> 4
- net /SWD_CLK: track 0.00 -> 35.5 mm, vias 0 -> 2
- net Net-(J4-SWO): track 0.00 -> 28.6 mm, vias 0 -> 2
- net +5V: track 0.00 -> 20.0 mm, vias 0 -> 4
- net Net-(R6-Pad1): track 0.00 -> 16.6 mm
- net /SMPS_FB: track 0.00 -> 15.6 mm, vias 0 -> 2
- net /UART_RXC: track 0.00 -> 12.4 mm
- net /LSE_IN: track 0.00 -> 12.1 mm, vias 0 -> 2
- net /RF: track 0.00 -> 11.7 mm, vias 0 -> 2
- net /UART_TXC: track 0.00 -> 11.0 mm
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- added copper zone on In2.Cu, net +3V3
- added copper zone on In2.Cu, net +5V
- added copper zone on In1.Cu, net GND
Other:
- board size 65 x 56 mm -> 60 x 16.5 mm
- copper layers 2 -> 4
- rule pad_to_mask_clearance: 0 -> 0.8
- board text removed: "${ISSUE_DATE}"
- board text removed: "0"
- board text removed: "0 mm"
- board text removed: "0.01 mm"
- board text removed: "0.02"
- board text removed: "0.035 mm"
- board text removed: "0.2000 mm / 0.0000 mm"
- board text removed: "0.3000 mm"
- board text removed: "1"
- board text removed: "1.51 mm"
- board text removed: "1.6000 mm"
- board text removed: "2"
- board text removed: "3.3"
- board text removed: "4.5"
- board text removed: "65.0000 mm x 56.0000 mm"
- board text removed: "B.Cu"
- board text removed: "B.Mask"
- board text removed: "B.Paste"
- board text removed: "B.Silkscreen"
- board text removed: "BOARD CHARACTERISTICS"
- board text removed: "Board Thickness:"
- board text removed: "Board overall dimensions:"
- board text removed: "Bottom Silk Screen"
- board text removed: "Bottom Solder Mask"
- board text removed: "Bottom Solder Paste"
- board text removed: "CAMERA (OPTIONAL)"
- board text removed: "Castellated pads:"
- board text removed: "Color"
- board text removed: "Copper Finish:"
- board text removed: "Copper Layer Count:"
- board text removed: "DISPLAY (OPTIONAL)"
- board text removed: "Dielectric"
- board text removed: "Edge card connectors:"
- board text removed: "Epsilon R"
- board text removed: "Extend PCB edge 0.5mm if using SMT header"
- board text removed: "F.Cu"
- board text removed: "F.Mask"
- board text removed: "F.Paste"
- board text removed: "F.Silkscreen"
- board text removed: "FR4"
- board text removed: "Green"
- board text removed: "Impedance Control:"
- board text removed: "Layer Name"
- board text removed: "Loss Tangent"
- board text removed: "Material"
- board text removed: "Min hole diameter:"
- board text removed: "Min track/spacing:"
- board text removed: "No"
- board text removed: "None"
- board text removed: "Not specified"
- board text removed: "Plated Board Edge:"
- board text removed: "PoE"
- board text removed: "RJ45"
- board text removed: "Thickness (mm)"
- board text removed: "Top Silk Screen"
- board text removed: "Top Solder Mask"
- board text removed: "Top Solder Paste"
- board text removed: "Type"
- board text removed: "USB"
- board text removed: "copper"
- board text removed: "core"

Commit message: Update 03
Project accomplished
Parts:
- added FID1: Fiducial, Fiducial:Fiducial_1mm_Mask2mm, F.Cu at (126.5, 49.0)
- added FID2: Fiducial, Fiducial:Fiducial_1mm_Mask2mm, F.Cu at (170.0, 49.0)
- added FID3: Fiducial, Fiducial:Fiducial_1mm_Mask2mm, F.Cu at (170.0, 68.5)
- added H1: MountingHole_Pad, MountingHole:MountingHole_2.2mm_M2_Pad, F.Cu at (174.5, 50.5)
- added H2: MountingHole_Pad, MountingHole:MountingHole_2.2mm_M2_Pad, F.Cu at (174.5, 67.0)
- added H3: MountingHole_Pad, MountingHole:MountingHole_2.2mm_M2_Pad, F.Cu at (122.5, 67.0)
- added H4: MountingHole_Pad, MountingHole:MountingHole_2.2mm_M2_Pad, F.Cu at (122.5, 50.5)
- moved J1 7.35 mm to (145.4, 62.0), turned to 0 degrees
- moved C13 5.18 mm to (141.6, 59.6)
- moved D1 2.97 mm to (159.9, 64.1)
- moved R3 2.97 mm to (159.9, 66.3)
- moved C10 2.90 mm to (133.9, 66.1)
- moved C11 2.90 mm to (133.9, 64.6)
- moved C19 2.90 mm to (139.4, 66.1)
- moved R2 2.90 mm to (157.0, 61.3)
- moved R7 2.90 mm to (139.4, 64.6)
- moved X1 2.90 mm to (166.4, 65.1)
- moved C1 2.90 mm to (148.4, 53.6)
- moved C14 2.90 mm to (163.4, 51.6)
- moved C15 2.90 mm to (169.6, 58.1)
- moved C16 2.90 mm to (169.6, 61.1)
- moved C17 2.90 mm to (157.4, 51.6)
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Routing:
- net /BOOT: track 9.20 -> 26.6 mm
- net /SWD_NRST: track 42.1 -> 30.6 mm, vias 4 -> 2
- net +3V3: track 68.9 -> 58.6 mm, vias 15 -> 16
- net Net-(X1-Pad2): track 7.98 -> 6.01 mm
- net /SMPS_FB: track 15.6 -> 13.8 mm
- net /USB_D-: track 42.7 -> 40.9 mm
- net /UART_RXC: track 12.4 -> 10.7 mm
- net /USBC_D-: track 8.30 -> 9.83 mm
- net /SMPSLX: track 5.90 -> 4.55 mm
- net /UART_TXC: track 11.0 -> 12.2 mm
- net /USB_D+: track 47.4 -> 46.4 mm
- net /SMPSLXL: track 1.54 -> 2.48 mm
- net Net-(R6-Pad1): track 16.6 -> 15.7 mm
- net GND: track 82.1 -> 82.9 mm, vias 41 -> 30
- net /RF: track 11.7 -> 12.3 mm
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Other:
- board size 60 x 16.5 mm -> 60 x 22.5 mm
- rule pad_to_mask_clearance: 0.8 -> 0
- board text added: "02-24-2024"
- board text added: "BOOT"
- board text added: "DJAMAL ZILAL"
- board text added: "RF"
- board text added: "STM32WB - Rev01"
- board text added: "SWD"
- board text added: "UART"
- board text added: "USB"

Commit message: Update 4
Errors fixed
Routing:
- net /UART_TX: track 4.69 -> 7.97 mm
- net Net-(X1-Pad2): track 6.01 -> 8.34 mm
- net +3V3: track 58.6 -> 60.5 mm
- net +5V: track 19.8 -> 18.7 mm
- net /USB_D-: track 40.9 -> 41.8 mm
- net /SMPSLX: track 4.55 -> 5.07 mm
